File: headphone_sum.kicad_sch (KiCad schematic)
At the start: 42 parts, among them J1 IN_L1, J2 IN_L2, J3 IN_R1, J4 IN_R2, J5 OUT_LR, J6 Eurorack Power, J7 Conn_01x03_Male, J8 Conn_01x02_Female, U1 TL072, U2 NE5532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

Commit message: Remove duplicate front/back file, old KiCad files.
Parts:
- added R15, R16: 200k, Resistor_SMD:R_0603_1608Metric_Pad0.98x0.95mm_HandSolder, symbol Device:R
Connections:
- net R_IN: now also R16.2
- net at C12.2, C13.1, R8.1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: no longer J3.TN
- net at C12.1, R1.1, R2.1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: now also R16.1
- net at C11.1, R5.1, R6.1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: now also R15.1
- net at J2.T, R2.2: now also R15.2
- no-connect marks 5 -> 6
Other:
- note added: "https://www.falstad.com/circuit/circuitjs.html?ctz=CQAgjCAMB0l5YCsA2ATIkAWR0DsZNN8BmVZADgE5JKRFc67I6BTAWjDACgA3ED5M0rJ+YQeBHMIhZrKhRoiLgHNR44WqlhU8yFwBOmif2SZjU+HAMhyU1ORCpUZ7Q+aZi8LgHdHz8PZ+LriSXACGNlIhQeDRDkiiGGCWcKxspGYWllwA8jFg0fbx0bJcAMaRIKYx1e547JwgxNDEuPTsxGC0MHDcvrZVZgOuUD41Zk4ugXqqw5Q6A6iQbqOGAlLibNVicsnZquuOmMyH6JKjfKfHRjvyEANysorWHNHEiDpsA+86WV4HBREHk+gKwmBWekuoOBojeHzu4E4j10zzWt0w1S2Z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"
- moved on the sheet: R2, R5

Commit message: BOM and position file fixes
Parts:
- R15, R16: LCSC C25803 -> C25811; LCSC part number C25803 -> C25811
Changed lines of the file:
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@@
       (effects (font (size 1.27 1.27)) hide)
     )
-    (property "LCSC part number" "C25803" (at 50.8 80.01 0)
-      (effects (font (size 1.27 1.27)) hide)
-    )
-    (property "LCSC" "C25803" (at 50.8 80.01 0)
+    (property "LCSC part number" "C25811" (at 50.8 80.01 0)
+      (effects (font (size 1.27 1.27)) hide)
+    )
+    (property "LCSC" "C25811" (at 50.8 80.01 0)
       (effects (font (size 1.27 1.27)) hide)
     )
@@
       (effects (font (size 1.27 1.27)) hide)
     )
-    (property "LCSC part number" "C25803" (at 50.8 57.15 0)
-      (effects (font (size 1.27 1.27)) hide)
-    )
-    (property "LCSC" "C25803" (at 50.8 57.15 0)
-      (effects (font (size 1.27 1.27)) hide)
-    )
+    (property "LCSC part number" "C25811" (at 50.8 57.15 0)
+      (effects (font (size 1.27 1.27)) hide)
+    )
+    (property "LCSC" "C25811" (at 50.8 57.15 0)
+      (effects (font (size 1.27 1.27)) hide)
+    )

Commit message: v1.1.1, fix some LCSC part numbers, fix D1,D2 footprint
Parts:
- D1, D2: footprint Diode_SMD:D_SOD-523 -> Diode_SMD:D_SOD-323
Changed lines of the file:
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@@
       (effects (font (size 1.27 1.27)))
     )
-    (property "Footprint" "Diode_SMD:D_SOD-523" (at 44.45 160.655 0)
+    (property "Footprint" "Diode_SMD:D_SOD-323" (at 44.45 160.655 0)
       (effects (font (size 1.27 1.27)) hide)
     )
@@
       (effects (font (size 1.27 1.27)))
     )
-    (property "Footprint" "Diode_SMD:D_SOD-523" (at 44.45 189.865 0)
+    (property "Footprint" "Diode_SMD:D_SOD-323" (at 44.45 189.865 0)
       (effects (font (size 1.27 1.27)) hide)
     )
